File: hardware/pcb/10KeyMacropad.kicad_pcb (KiCad board)
At the start: 2 copper layers, 62 x 98 mm, 18 parts, among them SW1 SW_Push, SW10 SW_Push, SW2 SW_Push, SW3 SW_Push, SW4 SW_Push, SW5 SW_Push, SW6 SW_Push, SW7 SW_Push, SW8 SW_Push, SW9 SW_Push

Commit message: Fixed PCB to use non hotswappable switches
Parts:
- SW1, SW10, SW2, SW3, SW4, SW5, SW6, SW7, SW8, SW9: footprint MX_Hotswap:MX-Hotswap-1U -> Button_Switch_Keyboard:SW_Cherry_MX_1.00u_PCB
- moved SW1 5.59 mm to (129.5, 35.0)
- moved SW10 5.59 mm to (148.5, 111.0)
- moved SW2 5.59 mm to (129.5, 54.0)
- moved SW3 5.59 mm to (129.5, 73.0)
- moved SW4 5.59 mm to (129.5, 92.0)
- moved SW5 5.59 mm to (129.5, 111.0)
- moved SW6 5.59 mm to (148.5, 35.0)
- moved SW7 5.59 mm to (148.5, 54.0)
- moved SW8 5.59 mm to (148.5, 73.0)
- moved SW9 5.59 mm to (148.5, 92.0)
Routing:
- net GND: track 358.2 -> 400.8 mm
- net Net-(A1-GPIO4): track 67.5 -> 72.0 mm
- net Net-(A1-GPIO5): track 94.8 -> 98.3 mm
- net Net-(A1-GPIO10): track 97.1 -> 100.5 mm
- net Net-(A1-GPIO9): track 74.9 -> 78.3 mm
- net Net-(A1-GPIO3): track 38.1 -> 41.6 mm
- net Net-(A1-GPIO2): track 23.7 -> 27.1 mm
- net Net-(A1-GPIO6): track 46.8 -> 50.1 mm
- net Net-(A1-GPIO7): track 69.4 -> 72.5 mm
- net Net-(A1-GPIO1): track 10.7 -> 13.4 mm
